File: hardware/project/ETH6C16MUX/Connector.sch (KiCad schematic (older format))
At the start: 1 part

Commit message: Schematic design
Parts:
- added J801: 615008145221, ETH6C16MXU:615008145221, symbol Connector:RJ45_Shielded
- J802: renamed from J?; footprint (none) -> ETH6C16MXU:Socket_DIN41612-CaseC1-AC-Male-64Pin-2rows
Connections:
- wire segments 60 -> 65
- no-connect marks 36 -> 40
Changed lines of the file:
@@
 $Descr A4 11693 8268
 encoding utf-8
-Sheet 8 8
+Sheet 8 9
 Title ""
 Date ""
@@
 $EndDescr
 $Comp
-L Connector:C64AC J?
+L Connector:C64AC J802
 U 1 1 5DB3A84B
 P 5950 4000
-F 0 "J?" H 6130 4096 50  0000 L CNN
+F 0 "J802" H 6130 4096 50  0000 L CNN
 F 1 "C64AC" H 6130 4005 50  0000 L CNN
-F 2 "" H 5950 4050 50  0001 C CNN
+F 2 "ETH6C16MXU:Socket_DIN41612-CaseC1-AC-Male-64Pin-2rows" H 5950 4050 50  0001 C CNN
 F 3 " ~" H 5950 4050 50  0001 C CNN
 	1    5950 4000
@@
 	5600 6200 5600 6100
 $Comp
-L power:+24V #PWR?
+L power:+24V #PWR0805
 U 1 1 5D7D1F7C
 P 5550 7100
-F 0 "#PWR?" H 5550 6950 50  0001 C CNN
+F 0 "#PWR0805" H 5550 6950 50  0001 C CNN
 F 1 "+24V" V 5565 7228 50  0000 L CNN
 F 2 "" H 5550 7100 50  0001 C CNN
@@
 Connection ~ 5600 7100
 $Comp
-L power:GND #PWR?
+L power:GND #PWR0804
 U 1 1 5D7D46BE
 P 5550 6300
-F 0 "#PWR?" H 5550 6050 50  0001 C CNN
+F 0 "#PWR0804" H 5550 6050 50  0001 C CNN
 F 1 "GND" V 5555 6172 50  0000 R CNN
 F 2 "" H 5550 6300 50  0001 C CNN
@@
 Wire Wire Line
 	5600 5000 5650 5000
-Text HLabel 5550 4700 0    50   BiDi ~ 0
+Text HLabel 5300 4700 0    50   BiDi ~ 0
 TX+
-Text HLabel 5550 4900 0    50   BiDi ~ 0
+Text HLabel 5300 4900 0    50   BiDi ~ 0
 TX-
-Text HLabel 5550 4600 0    50   BiDi ~ 0
+Text HLabel 5300 4600 0    50   BiDi ~ 0
 RX+
-Text HLabel 5550 4800 0    50   BiDi ~ 0
+Text HLabel 5300 4800 0    50   BiDi ~ 0
 RX-
-Wire Wire Line
-	5550 4900 5650 4900
-Wire Wire Line
-	5550 4800 5650 4800
-Wire Wire Line
-	5550 4700 5650 4700
-Wire Wire Line
-	5550 4600 5650 4600
-$Comp
-L power:Earth #PWR?
+$Comp
+L power:Earth #PWR0803
 U 1 1 5D7F1666
 P 5550 5050
-F 0 "#PWR?" H 5550 4800 50  0001 C CNN
+F 0 "#PWR0803" H 5550 4800 50  0001 C CNN
 F 1 "Earth" H 5550 4900 50  0001 C CNN
 F 2 "" H 5550 5050 50  0001 C CNN
@@
 	5600 5050 5600 5000
 $Comp
-L power:Earth #PWR?
+L power:Earth #PWR0802
 U 1 1 5D7F6C0C
 P 5550 4250
-F 0 "#PWR?" H 5550 4000 50  0001 C CNN
+F 0 "#PWR0802" H 5550 4000 50  0001 C CNN
 F 1 "Earth" H 5550 4100 50  0001 C CNN
 F 2 "" H 5550 4250 50  0001 C CNN
@@
 Text HLabel 5550 3050 0    50   BiDi ~ 0
 F
+$Comp
+L Connector:RJ45_Shielded J801
+U 1 1 5E56A100
+P 1350 1550
+F 0 "J801" H 1350 2200 50  0000 C CNN
+F 1 "615008145221" H 1350 2100 50  0000 C CNN
+F 2 "ETH6C16MXU:615008145221" V 1350 1575 50  0001 C CNN
+F 3 "~" V 1350 1575 50  0001 C CNN
+	1    1350 1550
+	1    0    0    -1
+$EndComp
+NoConn ~ 1750 1150
+NoConn ~ 1750 1250
+NoConn ~ 1750 1450
+NoConn ~ 1750 1550
+Wire Wire Line
+	5300 4900 5650 4900
+Wire Wire Line
+	5300 4800 5650 4800
+Wire Wire Line
+	5300 4700 5650 4700
+Wire Wire Line
+	5300 4600 5650 4600
+Text Label 5350 4600 0    50   ~ 0
+RX+
+Text Label 5350 4700 0    50   ~ 0
+TX+
+Text Label 5350 4800 0    50   ~ 0
+RX-
+Text Label 5350 4900 0    50   ~ 0
+TX-
+Text Label 2050 1650 2    50   ~ 0
+RX+
+Text Label 2050 1850 2    50   ~ 0
+TX+
+Text Label 2050 1350 2    50   ~ 0
+RX-
+Text Label 2050 1750 2    50   ~ 0
+TX-
+Wire Wire Line
+	2050 1350 1750 1350
+Wire Wire Line
+	1750 1650 2050 1650
+Wire Wire Line
+	1750 1750 2050 1750
+Wire Wire Line
+	1750 1850 2050 1850
+$Comp
+L power:Earth #PWR0801
+U 1 1 5E5917B7
+P 1350 2100
+F 0 "#PWR0801" H 1350 1850 50  0001 C CNN
+F 1 "Earth" H 1350 1950 50  0001 C CNN
+F 2 "" H 1350 2100 50  0001 C CNN
+F 3 "~" H 1350 2100 50  0001 C CNN
+	1    1350 2100
+	1    0    0    -1
+$EndComp
+Wire Wire Line
+	1350 2100 1350 2050
 $EndSCHEMATC

Commit message: PCB design, need to redesign of the board to board connectors.
Parts:
- removed J801: 615008145221, ETH6C16MXU:615008145221, symbol Connector:RJ45_Shielded
- added J802: Conn_01x06, symbol Connector_Generic:Conn_01x06
- renumbered J802 to J801
Connections:
- wire segments 65 -> 66
- no-connect marks 40 -> 36
Changed lines of the file:
@@
 $EndDescr
 $Comp
-L Connector:C64AC J802
+L Connector:C64AC J801
 U 1 1 5DB3A84B
 P 5950 4000
-F 0 "J802" H 6130 4096 50  0000 L CNN
+F 0 "J801" H 6130 4096 50  0000 L CNN
 F 1 "C64AC" H 6130 4005 50  0000 L CNN
 F 2 "ETH6C16MXU:Socket_DIN41612-CaseC1-AC-Male-64Pin-2rows" H 5950 4050 50  0001 C CNN
@@
 NoConn ~ 5650 1300
 NoConn ~ 5650 1200
-Wire Wire Line
-	5600 1050 5550 1050
 Connection ~ 5600 1050
 Wire Wire Line
 	5600 1050 5600 1100
-Wire Wire Line
-	5600 1450 5550 1450
 Connection ~ 5600 1450
 Wire Wire Line
 	5600 1450 5600 1500
-Wire Wire Line
-	5600 1850 5550 1850
 Connection ~ 5600 1850
 Wire Wire Line
 	5600 1850 5600 1900
-Wire Wire Line
-	5600 2250 5550 2250
 Connection ~ 5600 2250
 Wire Wire Line
 	5600 2250 5600 2300
-Wire Wire Line
-	5600 2650 5550 2650
 Connection ~ 5600 2650
 Wire Wire Line
 	5600 2650 5600 2700
-Wire Wire Line
-	5600 3050 5550 3050
 Connection ~ 5600 3050
 Wire Wire Line
 	5600 3050 5600 3100
-Text HLabel 5550 1050 0    50   BiDi ~ 0
+Text HLabel 5300 1050 0    50   BiDi ~ 0
 A
-Text HLabel 5550 1450 0    50   BiDi ~ 0
+Text HLabel 5300 1450 0    50   BiDi ~ 0
 B
-Text HLabel 5550 1850 0    50   BiDi ~ 0
+Text HLabel 5300 1850 0    50   BiDi ~ 0
 C
-Text HLabel 5550 2250 0    50   BiDi ~ 0
+Text HLabel 5300 2250 0    50   BiDi ~ 0
 D
-Text HLabel 5550 2650 0    50   BiDi ~ 0
+Text HLabel 5300 2650 0    50   BiDi ~ 0
 E
-Text HLabel 5550 3050 0    50   BiDi ~ 0
+Text HLabel 5300 3050 0    50   BiDi ~ 0
 F
-$Comp
-L Connector:RJ45_Shielded J801
-U 1 1 5E56A100
-P 1350 1550
-F 0 "J801" H 1350 2200 50  0000 C CNN
-F 1 "615008145221" H 1350 2100 50  0000 C CNN
-F 2 "ETH6C16MXU:615008145221" V 1350 1575 50  0001 C CNN
-F 3 "~" V 1350 1575 50  0001 C CNN
-	1    1350 1550
-	1    0    0    -1
-$EndComp
-NoConn ~ 1750 1150
-NoConn ~ 1750 1250
-NoConn ~ 1750 1450
-NoConn ~ 1750 1550
 Wire Wire Line
 	5300 4900 5650 4900
@@
 Text Label 5350 4900 0    50   ~ 0
 TX-
-Text Label 2050 1650 2    50   ~ 0
-RX+
-Text Label 2050 1850 2    50   ~ 0
-TX+
-Text Label 2050 1350 2    50   ~ 0
-RX-
-Text Label 2050 1750 2    50   ~ 0
-TX-
-Wire Wire Line
-	2050 1350 1750 1350
-Wire Wire Line
-	1750 1650 2050 1650
-Wire Wire Line
-	1750 1750 2050 1750
-Wire Wire Line
-	1750 1850 2050 1850
-$Comp
-L power:Earth #PWR0801
-U 1 1 5E5917B7
-P 1350 2100
-F 0 "#PWR0801" H 1350 1850 50  0001 C CNN
-F 1 "Earth" H 1350 1950 50  0001 C CNN
-F 2 "" H 1350 2100 50  0001 C CNN
-F 3 "~" H 1350 2100 50  0001 C CNN
-	1    1350 2100
-	1    0    0    -1
-$EndComp
-Wire Wire Line
-	1350 2100 1350 2050
+Wire Wire Line
+	5300 3050 5600 3050
+Wire Wire Line
+	5300 2650 5600 2650
+Wire Wire Line
+	5300 2250 5600 2250
+Wire Wire Line
+	5300 1850 5600 1850
+Wire Wire Line
+	5300 1450 5600 1450
+Wire Wire Line
+	5300 1050 5600 1050
+Text Label 5350 1050 0    50   ~ 0
+A
+Text Label 5350 1450 0    50   ~ 0
+B
+Text Label 5350 1850 0    50   ~ 0
+C
+Text Label 5350 2250 0    50   ~ 0
+D
+Text Label 5350 2650 0    50   ~ 0
+E
+Text Label 5350 3050 0    50   ~ 0
+F
+Text Label 3650 1000 2    50   ~ 0
+A
+Text Label 3650 1100 2    50   ~ 0
+B
+Text Label 3650 1200 2    50   ~ 0
+C
+Text Label 3650 1300 2    50   ~ 0
+D
+Text Label 3650 1400 2    50   ~ 0
+E
+Text Label 3650 1500 2    50   ~ 0
+F
+$Comp
+L Connector_Generic:Conn_01x06 J802
+U 1 1 61D03557
+P 3200 1200
+F 0 "J802" H 3118 1617 50  0000 C CNN
+F 1 "Conn_01x06" H 3118 1526 50  0000 C CNN
+F 2 "" H 3200 1200 50  0001 C CNN
+F 3 "~" H 3200 1200 50  0001 C CNN
+	1    3200 1200
+	-1   0    0    -1
+$EndComp
+Wire Wire Line
+	3400 1000 3650 1000
+Wire Wire Line
+	3400 1100 3650 1100
+Wire Wire Line
+	3400 1200 3650 1200
+Wire Wire Line
+	3400 1300 3650 1300
+Wire Wire Line
+	3400 1400 3650 1400
+Wire Wire Line
+	3400 1500 3650 1500
 $EndSCHEMATC
