File: hardware/project/ETH6C16MUX/ETH6C16MUX.kicad_pcb (KiCad board)
At the start: 2 copper layers, 160 x 100 mm, 210 parts, among them J301 Conn_02x05, J302 Conn_02x01, J303 Conn_02x01, J501 105133-0001, J601 1-103673-5, J801 C64AC, J901 IPT1-110-01-L-D-VS, K601 HE3621A0500, K602 HE3621A0500, K603 HE3621A0500, K604 HE3621A0500, K605 HE3621A0500, K606 HE3621A0500, K607 HE3621A0500, K608 HE3621A0500, K609 HE3621A0500, K610 HE3621A0500, K611 HE3621A0500, K612 HE3621A0500, K613 HE3621A0500, K614 HE3621A0500, K615 HE3621A0500, K616 HE3621A0500, K617 HE3621A0500, K618 HE3621A0500, K619 HE3621A0500, K620 HE3621A0500, K621 HE3621A0500, K622 HE3621A0500, K623 HE3621A0500, K624 HE3621A0500, K625 HE3621A0500, K626 HE3621A0500, K627 HE3621A0500, K628 HE3621A0500, K629 HE3621A0500, K630 HE3621A0500, K631 HE3621A0500, K632 HE3621A0500, K633 HE3621A0500, K634 HE3621A0500, K635 HE3621A0500, K636 HE3621A0500, K637 HE3621A0500, K638 HE3621A0500, K639 HE3621A0500, K640 HE3621A0500, K641 HE3621A0500, K642 HE3621A0500, K643 HE3621A0500, K644 HE3621A0500, K645 HE3621A0500, K646 HE3621A0500, K647 HE3621A0500, K648 HE3621A0500, K649 HE3621A0500, K650 HE3621A0500, K651 HE3621A0500, K652 HE3621A0500, K653 HE3621A0500, K654 HE3621A0500, Q701 IRFR5410, U201 LC03-3.3, U202 LAN8742, U203 LC03-3.3, U204 SR3.3, U205 SR3.3, U206 ASDM1-50.000MHZ-LC-T, U301 ASDM1-20.000MHZ-LC-T, U302 S25FL064L_SOIC, U303 S25FL064L_SOIC, U304 STM32F765ZGT6, U305 MCP9804, U401 iCE40-HX4K-TQ144, U402 ASDM1-100.000MHZ-LC-T, U501 FT230XQ, U502 824011, U601 ULN2803A, U602 ULN2803A, U603 ULN2803A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

Commit message: PCB layout, board to board connector changed.
Parts:
- removed H901, H902: MountingHole, MountingHole:MountingHole_3mm_Pad
- removed J901: IPT1-110-01-L-D-VS, Connector_PinHeader_2.54mm:PinHeader_2x10_P2.54mm_Vertical_SMD
- added H101: MountingHole, MountingHole:MountingHole_3.2mm_M3_DIN965_Pad, F.Cu at (66.0, 104.0)
- added H102: MountingHole, MountingHole:MountingHole_3.2mm_M3_DIN965_Pad, F.Cu at (66.0, 47.0)
- added J801: Conn_01x06, Connector_PinSocket_2.54mm:PinSocket_1x06_P2.54mm_Vertical, F.Cu at (204.0, 55.0)
- added J802: Conn_02x09_Odd_Even, Connector_PinSocket_2.54mm:PinSocket_2x09_P2.54mm_Vertical, F.Cu at (83.0, 115.0)
- moved J303 278.8 mm to (170.0, 134.1), turned to 90 degrees
- moved J302 27.3 mm to (152.0, 152.0), turned to 90 degrees
- moved C705 4.51 mm to (169.2, 128.8)
- moved FB702 4.51 mm to (173.0, 127.3)
- moved C710 4.51 mm to (173.0, 130.4)
- moved C703 4.00 mm to (176.8, 123.0)
- moved C704 4.00 mm to (170.4, 116.1)
- moved C708 4.00 mm to (176.5, 118.7)
- moved C709 4.00 mm to (170.4, 116.1)
- moved FB701 4.00 mm to (177.3, 129.1)
- moved U703 4.00 mm to (170.4, 122.2)
- moved U607 3.51 mm to (157.7, 97.9)
- moved U601 2.83 mm to (143.5, 97.9)
- moved U603 2.83 mm to (143.5, 97.9)
- moved D303 2.62 mm to (64.5, 121.0)
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- renumbered C706 to C704, C707 to C705, C704 to C706, C705 to C707, J801 to J803, L502 to L501, U704 to U703, U703 to U704
Connections:
- net /FPGA/MCU_SPI3_MISO renamed /Connector/MCU_SPI3_MISO
- net /FPGA/MCU_SPI3_MOSI renamed /Connector/MCU_SPI3_MOSI
- net /FPGA/MCU_SPI3_SCLK renamed /Connector/MCU_SPI3_SCLK
- U304 pad 1: /MCU/FPGA2_SPI4_SLCK -> /Connector/FPGA2_SPI4_SLCK
- U304 pad 3: /MCU/FPGA2_SPI4_CS -> /Connector/FPGA2_SPI4_CS
- U304 pad 4: /MCU/FPGA2_SPI4_MISO -> /Connector/FPGA2_SPI4_MISO
- U304 pad 46: /MCU/MODULE_DETECT -> /Connector/MODULE_DETECT
- U304 pad 5: /MCU/FPGA2_SPI4_MOSI -> /Connector/FPGA2_SPI4_MOSI
- U304 pad 65: /MCU/FPGA2_CDONE -> /Connector/FPGA2_CDONE
- U304 pad 66: /MCU/FPGA2_CRESET_B -> /Connector/FPGA2_CRESET_B
- U304 pad 67: /MCU/FPGA2_CBSEL0 -> /Connector/FPGA2_CBSEL0
- U304 pad 68: /MCU/FPGA2_CBSEL1 -> /Connector/FPGA2_CBSEL1
- U304 pad 96: /MCU/FPGA2_CFG_CS -> /Connector/FPGA2_CFG_CS

Commit message: PCB layout, deleted USB.
Parts:
- removed C501, C502: 22u, ETH6C16MXU:C_1210_BB_3225Metric_Pad1.42x2.65mm_HandSolder
- removed C503, C505: 1u, ETH6C16MXU:C_0603_B_Pad1.05x0.95mm_HandSolder
- removed C504: 100n, ETH6C16MXU:C_0603_A_Pad1.05x0.95mm_HandSolder
- removed D501: CUS08F30, Diode_SMD:D_SOD-323_HandSoldering
- removed FB501: 742792031, ETH6C16MXU:R_0805_D_Pad1.15x1.40mm_HandSolder
- removed J601: 1-103673-5, ETH6C16MXU:1-103673-5
- removed K601, K602, K603: HE3621A0500, ETH6C16MXU:HE360_x-5331272-5
- removed L501: 744233121, ETH6C16MXU:744233121
- removed R501: 0, Resistor_SMD:R_0612_1632Metric_Pad1.18x3.40mm_HandSolder
- removed R502, R503: 27, Resistor_SMD:R_0603_1608Metric_Pad1.05x0.95mm_HandSolder
- removed R504: 10k, ETH6C16MXU:R_0603_E_Pad1.05x0.95mm_HandSolder
- removed the U502 at (137.9, 125.1)
- removed the U601 at (143.5, 97.9)
- removed the U604 at (129.4, 97.9)
- added C411: 1u, ETH6C16MXU:C_0603_B_Pad1.05x0.95mm_HandSolder, B.Cu at (119.8, 133.6)
- added C412: 1u, ETH6C16MXU:C_0603_B_Pad1.05x0.95mm_HandSolder, B.Cu at (120.5, 117.1)
- added C413: 1u, ETH6C16MXU:C_0603_B_Pad1.05x0.95mm_HandSolder, B.Cu at (121.9, 126.6)
- added C414: 1u, ETH6C16MXU:C_0603_B_Pad1.05x0.95mm_HandSolder, B.Cu at (121.9, 122.6)
- added K501: HE3621A0500, ETH6C16MXU:HE360_x-5331272-5, F.Cu at (76.6, 98.3)
- added K502: HE3621A0500, ETH6C16MXU:HE360_x-5331272-5, F.Cu at (81.8, 98.3)
- added K503: HE3621A0500, ETH6C16MXU:HE360_x-5331272-5, F.Cu at (87.0, 98.3)
- added U504: ULN2803A, Package_SO:SOIC-18W_7.5x11.6mm_P1.27mm, B.Cu at (129.5, 99.2)
- C211, C212, C304, C305, C310, C311, C312, C313, C314, C315, C316, C317, C318, C319, C320, C321, C322, C406, C407, C408, C409, C410, D401, FB301, FB302, R206, R207, R302, R309, R310, R311, R312, R403: moved to B.Cu
- C606: renamed from C706; moved to B.Cu
- C607: renamed from C707; moved to B.Cu
- J501: value 105133-0001 -> Conn_02x08_Counter_Clockwise; footprint Connector_USB:USB_Micro-B_Molex-105133-0001 -> Connector_IDC:IDC-Header_2x08_P2.54mm_Horizontal_Lock
- R603: renamed from R703; moved to B.Cu
- U204, U205: footprint Package_TO_SOT_SMD:SOT-143_Handsoldering -> Package_TO_SOT_SMD:SOT-143; moved to B.Cu
- U501: value FT230XQ -> ULN2803A; footprint Package_DFN_QFN:QFN-16-1EP_4x4mm_P0.65mm_EP2.1x2.1mm -> Package_SO:SOIC-18W_7.5x11.6mm_P1.27mm
- moved U402 499.0 mm to (97.2, 130.3)
- moved C405 497.4 mm to (94.7, 130.3), turned to 90 degrees
- moved R404 491.5 mm to (99.1, 126.4), turned to 180 degrees
- moved R402 486.7 mm to (99.7, 130.2), turned to 270 degrees
- moved C404 482.6 mm to (97.9, 123.6), turned to 270 degrees
- moved C403 482.3 mm to (99.8, 123.6), turned to 270 degrees
- moved C410 482.0 mm to (106.7, 133.6)
- moved R403 481.9 mm to (106.8, 131.2)
- moved C408 480.8 mm to (112.8, 133.6), turned to 180 degrees
- moved C406 478.6 mm to (106.7, 120.7)
- moved C409 475.3 mm to (106.7, 126.1)
- moved C407 471.5 mm to (108.6, 117.1), turned to 270 degrees
- moved C402 466.6 mm to (129.8, 124.6), turned to 270 degrees
- moved D401 463.4 mm to (123.1, 133.0), turned to 90 degrees
- moved C401 455.4 mm to (127.9, 124.6), turned to 270 degrees
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- renumbered C701 to C601, C702 to C602, C703 to C603, C704 to C604, C705 to C605, C708 to C608, C709 to C609, C710 to C610, D701 to D601, D702 to D602, D703 to D603, F701 to F601, FB701 to FB601, FB702 to FB602, J801 to J701, J802 to J702, J803 to J703, K604 to K504, K605 to K505, K606 to K506, K607 to K507, K608 to K508, K609 to K509, K610 to K510, K611 to K511, K612 to K512, K613 to K513, K614 to K514, K615 to K515, K616 to K516, K617 to K517, K618 to K518, K619 to K519, K620 to K520, K621 to K521, K622 to K522, K623 to K523, K624 to K524, K625 to K525, K626 to K526, K627 to K527, K628 to K528, K629 to K529, K630 to K530, K631 to K531, K632 to K532, K633 to K533, K634 to K534, K635 to K535, K636 to K536, K637 to K537, K638 to K538, K639 to K539, K640 to K540, K641 to K541, K642 to K542, K643 to K543, K644 to K544, K645 to K545, K646 to K546, K647 to K547, K648 to K548, K649 to K549, K650 to K550, K651 to K551, K652 to K552, K653 to K553, K654 to K554, Q701 to Q601, R701 to R601, R702 to R602, R704 to R604, R705 to R605, R706 to R606, U602 to U502, U603 to U503, U605 to U505, U606 to U506, U607 to U507, U701 to U601, U702 to U602, U703 to U603, U704 to U604
Connections:
- J501 pad 1: +5V_USB -> /Relays/PIN1
- J501 pad 2: /USB/F_USB_D- -> /Relays/PIN2
- J501 pad 3: /USB/F_USB_D+ -> /Relays/PIN3
- J501 pad 4: (no net) -> /Relays/PIN4
- J501 pad 5: GND -> /Relays/PIN5
- J501 pad 6: GND -> /Relays/PIN6
- J703 pad A10: /Connector/E -> (no net)
- J703 pad A12: /Connector/F -> (no net)
- J703 pad A3: (no net) -> /Connector/B
- J703 pad A4: /Connector/B -> /Connector/C
- J703 pad A5: (no net) -> /Connector/D
- J703 pad A6: /Connector/C -> /Connector/E
- J703 pad A7: (no net) -> /Connector/F
- J703 pad A8: /Connector/D -> (no net)
- J703 pad C10: /Connector/E -> (no net)
- J703 pad C12: /Connector/F -> (no net)
- J703 pad C3: (no net) -> /Connector/B
- J703 pad C4: /Connector/B -> /Connector/C
- J703 pad C5: (no net) -> /Connector/D
- J703 pad C6: /Connector/C -> /Connector/E
- J703 pad C7: (no net) -> /Connector/F
- J703 pad C8: /Connector/D -> (no net)
- U304 pad 69: /MCU/MCU_TX_UART3 -> (no net)
- U304 pad 70: /MCU/MCU_RX_UART3 -> (no net)
- U501 pad 1: Net-(C503-Pad1) -> /FPGA/RELAY0
- U501 pad 11: (no net) -> /Relays/RELAY8A
- U501 pad 12: (no net) -> /Relays/RELAY7A
- U501 pad 13: GND -> /Relays/RELAY6A
- U501 pad 14: (no net) -> /Relays/RELAY5A
- U501 pad 15: /MCU/MCU_RX_UART3 -> /Relays/RELAY4A
- U501 pad 16: (no net) -> /Relays/RELAY3A
- U501 pad 17: GND -> /Relays/RELAY2A
- U501 pad 2: /MCU/MCU_TX_UART3 -> /FPGA/RELAY1
- U501 pad 3: GND -> /FPGA/RELAY2
- U501 pad 4: (no net) -> /FPGA/RELAY3
- U501 pad 5: (no net) -> /FPGA/RELAY4
- U501 pad 6: /USB/USB_D- -> /FPGA/RELAY5
- U501 pad 7: /USB/USB_D+ -> /FPGA/RELAY6
- U501 pad 8: Net-(C503-Pad1) -> /FPGA/RELAY7
- U501 pad 9: Net-(C504-Pad1) -> GND

Commit message: Deleted FPGA part and change it for SPI IO chips. Change power supply circuit.
Parts:
- removed C319, C320, C321: 2u2, ETH6C16MXU:C_0805_C_Pad1.15x1.40mm_HandSolder
- removed the C401 at (127.9, 124.6)
- removed C406, C407, C408, C409, C411, C412, C413, C414: 1u, ETH6C16MXU:C_0603_B_Pad1.05x0.95mm_HandSolder
- removed C410: 100n, ETH6C16MXU:C_0603_A_Pad1.05x0.95mm_HandSolder
- removed the C602 at (195.5, 121.3)
- removed the C603 at (176.9, 123.9)
- removed the C604 at (170.5, 117.0)
- removed the C605 at (169.3, 129.7)
- removed the C606 at (90.5, 114.9)
- removed the C608 at (176.7, 119.6)
- removed the C609 at (170.6, 117.0)
- removed the C610 at (173.1, 131.3)
- removed D301: 551-0407, ETH6C16MXU:551-xx07
- removed D302: 551-0207, ETH6C16MXU:551-xx07
- removed D303: 551-0807, ETH6C16MXU:551-xx07
- removed the D401 at (123.1, 133.0)
- removed FB301, FB602: 742792031, ETH6C16MXU:R_0805_D_Pad1.15x1.40mm_HandSolder
- removed the FB601 at (177.4, 130.0)
- removed J702: Conn_02x09_Odd_Even, Connector_PinSocket_2.54mm:PinSocket_2x09_P2.54mm_Vertical
- removed the R401 at (128.5, 127.4)
- removed the R402 at (99.7, 130.2)
- removed the R403 at (106.8, 131.2)
- removed R404: 100, Resistor_SMD:R_0603_1608Metric_Pad1.05x0.95mm_HandSolder
- removed the R601 at (189.5, 131.0)
- removed the R605 at (183.6, 126.1)
- removed the R606 at (186.2, 126.2)
- removed the U204 at (181.4, 97.0)
- removed U205: SR3.3, Package_TO_SOT_SMD:SOT-143
- removed the U402 at (97.2, 130.3)
- removed U501, U502, U503, U504, U505, U506, U507: ULN2803A, Package_SO:SOIC-18W_7.5x11.6mm_P1.27mm
- removed the U601 at (185.2, 126.2)
- removed the U603 at (170.6, 123.1)
- removed the U604 at (91.7, 116.7)
- added D601: 150121M153000, ETH6C16MXU:150121M153000, F.Cu at (127.0, 130.0)
- added J502: Conn_02x08_Odd_Even, Connector_PinSocket_2.54mm:PinSocket_2x08_P2.54mm_Vertical, F.Cu at (118.0, 114.0)
- added M101: 60817-096, ETH6C16MXU:60817-096, F.Cu at (63.6, 134.4)
- added U301: MCZ33996, ETH6C16MXU:HSOP-32-1EP_7.5x11.0mm_P0.65mm_ThermalVias, F.Cu at (115.3, 98.8)
- added U302: MCZ33996, ETH6C16MXU:HSOP-32-1EP_7.5x11.0mm_P0.65mm_ThermalVias, F.Cu at (129.3, 98.9)
- added U303: MCZ33996, ETH6C16MXU:HSOP-32-1EP_7.5x11.0mm_P0.65mm_ThermalVias, F.Cu at (143.3, 98.9)
- added U304: MCZ33996, ETH6C16MXU:HSOP-32-1EP_7.5x11.0mm_P0.65mm_ThermalVias, F.Cu at (157.2, 98.9)
- added U403: LM1117MPX-3.3, Package_TO_SOT_SMD:SOT-223-3_TabPin2, F.Cu at (180.2, 124.7)
- C201, C202, C204, C205, C206, C207, C210, C213, C402, C405: footprint ETH6C16MXU:C_0603_A_Pad1.05x0.95mm_HandSolder -> Capacitor_SMD:C_0603_1608Metric_Pad1.05x0.95mm_HandSolder; moved to B.Cu
- C203, C209: footprint ETH6C16MXU:C_0603_B_Pad1.05x0.95mm_HandSolder -> Capacitor_SMD:C_0603_1608Metric_Pad1.05x0.95mm_HandSolder; moved to B.Cu
- C208, R201, R202, R203, R204, R205, R210: moved to B.Cu
- C403: value 10u -> 22u; footprint Capacitor_SMD:C_0805_2012Metric_Pad1.15x1.40mm_HandSolder -> Capacitor_SMD:C_1210_3225Metric_Pad1.42x2.65mm_HandSolder
- C404: value 100n -> 22u; footprint ETH6C16MXU:C_0603_A_Pad1.05x0.95mm_HandSolder -> Capacitor_SMD:C_1210_3225Metric_Pad1.42x2.65mm_HandSolder
- C601: renamed from C301; footprint ETH6C16MXU:C_0603_A_Pad1.05x0.95mm_HandSolder -> Capacitor_SMD:C_0603_1608Metric_Pad1.05x0.95mm_HandSolder
- C602: renamed from C302; footprint ETH6C16MXU:C_0603_A_Pad1.05x0.95mm_HandSolder -> Capacitor_SMD:C_0603_1608Metric_Pad1.05x0.95mm_HandSolder
- C603: renamed from C303; footprint ETH6C16MXU:C_0603_A_Pad1.05x0.95mm_HandSolder -> Capacitor_SMD:C_0603_1608Metric_Pad1.05x0.95mm_HandSolder
- C604: renamed from C304; footprint ETH6C16MXU:C_0805_C_Pad1.15x1.40mm_HandSolder -> Capacitor_SMD:C_0805_2012Metric_Pad1.15x1.40mm_HandSolder
- C605: renamed from C305; footprint ETH6C16MXU:C_0805_C_Pad1.15x1.40mm_HandSolder -> Capacitor_SMD:C_0805_2012Metric_Pad1.15x1.40mm_HandSolder
- C606: renamed from C306; footprint ETH6C16MXU:C_0603_A_Pad1.05x0.95mm_HandSolder -> Capacitor_SMD:C_0603_1608Metric_Pad1.05x0.95mm_HandSolder
- C607: value 22u -> 1u; footprint ETH6C16MXU:C_1210_BB_3225Metric_Pad1.42x2.65mm_HandSolder -> Capacitor_SMD:C_0603_1608Metric_Pad1.05x0.95mm_HandSolder
- C608: renamed from C307; footprint ETH6C16MXU:C_0603_A_Pad1.05x0.95mm_HandSolder -> Capacitor_SMD:C_0603_1608Metric_Pad1.05x0.95mm_HandSolder
- C609: renamed from C308; footprint ETH6C16MXU:C_0603_A_Pad1.05x0.95mm_HandSolder -> Capacitor_SMD:C_0603_1608Metric_Pad1.05x0.95mm_HandSolder
- C610: renamed from C309; footprint ETH6C16MXU:C_0603_A_Pad1.05x0.95mm_HandSolder -> Capacitor_SMD:C_0603_1608Metric_Pad1.05x0.95mm_HandSolder
- C611: renamed from C310; footprint ETH6C16MXU:C_0603_A_Pad1.05x0.95mm_HandSolder -> Capacitor_SMD:C_0603_1608Metric_Pad1.05x0.95mm_HandSolder
- C612: renamed from C311; footprint ETH6C16MXU:C_0603_A_Pad1.05x0.95mm_HandSolder -> Capacitor_SMD:C_0603_1608Metric_Pad1.05x0.95mm_HandSolder
- C613: renamed from C312; footprint ETH6C16MXU:C_0603_A_Pad1.05x0.95mm_HandSolder -> Capacitor_SMD:C_0603_1608Metric_Pad1.05x0.95mm_HandSolder
- C614: renamed from C313; footprint ETH6C16MXU:C_0603_A_Pad1.05x0.95mm_HandSolder -> Capacitor_SMD:C_0603_1608Metric_Pad1.05x0.95mm_HandSolder
- C615: renamed from C314; footprint ETH6C16MXU:C_0603_A_Pad1.05x0.95mm_HandSolder -> Capacitor_SMD:C_0603_1608Metric_Pad1.05x0.95mm_HandSolder
- C616: renamed from C315; footprint ETH6C16MXU:C_0603_A_Pad1.05x0.95mm_HandSolder -> Capacitor_SMD:C_0603_1608Metric_Pad1.05x0.95mm_HandSolder
- C617: renamed from C316; footprint ETH6C16MXU:C_0603_A_Pad1.05x0.95mm_HandSolder -> Capacitor_SMD:C_0603_1608Metric_Pad1.05x0.95mm_HandSolder
- C618: renamed from C317; footprint ETH6C16MXU:C_0603_A_Pad1.05x0.95mm_HandSolder -> Capacitor_SMD:C_0603_1608Metric_Pad1.05x0.95mm_HandSolder
- C619: renamed from C318; footprint ETH6C16MXU:C_0603_A_Pad1.05x0.95mm_HandSolder -> Capacitor_SMD:C_0603_1608Metric_Pad1.05x0.95mm_HandSolder
- C620: renamed from C322; value 2u2 -> 1u; footprint ETH6C16MXU:C_0805_C_Pad1.15x1.40mm_HandSolder -> Capacitor_SMD:C_0603_1608Metric_Pad1.05x0.95mm_HandSolder
- FB201: footprint ETH6C16MXU:R_0805_D_Pad1.15x1.40mm_HandSolder -> Resistor_SMD:R_0805_2012Metric_Pad1.15x1.40mm_HandSolder; moved to B.Cu
- FB601: renamed from FB302; footprint ETH6C16MXU:R_0805_D_Pad1.15x1.40mm_HandSolder -> Resistor_SMD:R_0805_2012Metric_Pad1.15x1.40mm_HandSolder
- R208, R209: footprint ETH6C16MXU:R_0603_E_Pad1.05x0.95mm_HandSolder -> Resistor_SMD:R_0603_1608Metric_Pad1.05x0.95mm_HandSolder
- R211: moved to F.Cu
- R212, R213, R214: footprint ETH6C16MXU:R_0603_E_Pad1.05x0.95mm_HandSolder -> Resistor_SMD:R_0603_1608Metric_Pad1.05x0.95mm_HandSolder; moved to B.Cu
- R602: renamed from R302; footprint ETH6C16MXU:R_0603_E_Pad1.05x0.95mm_HandSolder -> Resistor_SMD:R_0603_1608Metric_Pad1.05x0.95mm_HandSolder
- R603: renamed from R303; moved to F.Cu
- R604: renamed from R304; moved to F.Cu
- R605: renamed from R305; footprint ETH6C16MXU:R_0603_E_Pad1.05x0.95mm_HandSolder -> Resistor_SMD:R_0603_1608Metric_Pad1.05x0.95mm_HandSolder
- R606: renamed from R306; value 270 -> 523; footprint ETH6C16MXU:R_0603_E_Pad1.05x0.95mm_HandSolder -> Resistor_SMD:R_0603_1608Metric_Pad1.05x0.95mm_HandSolder; moved to B.Cu
- R607: renamed from R307; value 270 -> 330; footprint ETH6C16MXU:R_0603_E_Pad1.05x0.95mm_HandSolder -> Resistor_SMD:R_0603_1608Metric_Pad1.05x0.95mm_HandSolder; moved to B.Cu
- R608: renamed from R308; value 270 -> 330; footprint ETH6C16MXU:R_0603_E_Pad1.05x0.95mm_HandSolder -> Resistor_SMD:R_0603_1608Metric_Pad1.05x0.95mm_HandSolder; moved to B.Cu
- R611: renamed from R311; footprint ETH6C16MXU:R_0603_E_Pad1.05x0.95mm_HandSolder -> Resistor_SMD:R_0603_1608Metric_Pad1.05x0.95mm_HandSolder
- R612: renamed from R312; footprint ETH6C16MXU:R_0603_E_Pad1.05x0.95mm_HandSolder -> Resistor_SMD:R_0603_1608Metric_Pad1.05x0.95mm_HandSolder
- U202: footprint Package_DFN_QFN:QFN-24-1EP_4x4mm_P0.5mm_EP2.6x2.6mm -> Package_DFN_QFN:QFN-24-1EP_4x4mm_P0.5mm_EP2.6x2.6mm_ThermalVias
- U401: value iCE40-HX4K-TQ144 -> TSR2-2450; footprint Package_QFP:TQFP-144_20x20mm_P0.5mm -> ETH6C16MXU:TSR2
- U602: renamed from U302; moved to F.Cu
- U603: renamed from U303; moved to F.Cu
- U605: renamed from U305; moved to F.Cu
- moved C209 299.2 mm to (169.8, 101.2), turned to 180 degrees
- moved R205 297.5 mm to (173.7, 100.3), turned to 270 degrees
- moved R212 296.5 mm to (169.8, 105.8)
- moved R208 296.2 mm to (176.0, 96.9), turned to 90 degrees
- moved R209 294.6 mm to (174.4, 96.9), turned to 90 degrees
- moved C202 293.0 mm to (169.8, 108.8)
- moved C203 292.8 mm to (175.3, 100.3), turned to 90 degrees
- moved C201 289.8 mm to (172.2, 109.3), turned to 90 degrees
- moved C213 289.3 mm to (169.8, 104.3), turned to 180 degrees
- moved C208 289.1 mm to (169.8, 102.7), turned to 180 degrees
- moved R201 286.6 mm to (184.2, 97.7), turned to 180 degrees
- moved C206 285.5 mm to (175.3, 109.3), turned to 270 degrees
- moved R213 284.8 mm to (169.8, 107.3)
- moved R214 283.8 mm to (173.7, 109.3), turned to 90 degrees
- moved R204 282.4 mm to (184.2, 107.1), turned to 180 degrees
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- renumbered C601 to C401, D601 to D401, D602 to D402, D603 to D403, F601 to F401, J501 to J301, J701 to J501, J703 to J503, J301 to J601, J302 to J602, J303 to J603, K501 to K301, K502 to K302, K503 to K303, K504 to K304, K505 to K305, K506 to K306, K507 to K307, K508 to K308, K509 to K309, K510 to K310, K511 to K311, K512 to K312, K513 to K313, K514 to K314, K515 to K315, K516 to K316, K517 to K317, K518 to K318, K519 to K319, K520 to K320, K521 to K321, K522 to K322, K523 to K323, K524 to K324, K525 to K325, K526 to K326, K527 to K327, K528 to K328, K529 to K329, K530 to K330, K531 to K331, K532 to K332, K533 to K333, K534 to K334, K535 to K335, K536 to K336, K537 to K337, K538 to K338, K539 to K339, K540 to K340, K541 to K341, K542 to K342, K543 to K343, K544 to K344, K545 to K345, K546 to K346, K547 to K347, K548 to K348, K549 to K349, K550 to K350, K551 to K351, K552 to K352, K553 to K353, K554 to K354, Q601 to Q401, R602 to R401, R603 to R402, R604 to R403, R301 to R601, R309 to R609, R310 to R610, U206 to U204, U602 to U402, U301 to U601, U304 to U604
Connections:
- net /Connector/MCU_SPI3_MISO renamed /MCU/MCU_SPI3_MISO
- C401 pad 1: Net-(C601-Pad1) -> Net-(C401-Pad1)
- C402 pad 1: Net-(C401-Pad1) -> +5V
- C402 pad 2: Net-(C401-Pad2) -> GND
- C403 pad 1: Net-(C403-Pad1) -> +5V
- C403 pad 2: Net-(C403-Pad2) -> GND
- C404 pad 1: Net-(C403-Pad1) -> +3V3
- C404 pad 2: Net-(C403-Pad2) -> GND
- C607 pad 1: +1.2V_FPGA_VCC -> Net-(C607-Pad1)
- C620 pad 1: /MCU/MCU_VREF+ -> /MCU/MCU_VDDA
- D401 pad 1: Net-(C601-Pad1) -> Net-(C401-Pad1)
- FB601 pad 1: /MCU/MCU_VREF+ -> /MCU/MCU_VDDA
- Q401 pad 2: Net-(C601-Pad1) -> Net-(C401-Pad1)
- R402 pad 1: Net-(C601-Pad1) -> Net-(C401-Pad1)
- R609 pad 1: Net-(R309-Pad1) -> Net-(C607-Pad1)
- U401 pad 1: /FPGA/RELAY27 -> Net-(C401-Pad1)
- U401 pad 2: /FPGA/RELAY28 -> GND
- U401 pad 3: /FPGA/RELAY29 -> +5V
- U402 pad 2: Net-(C601-Pad1) -> Net-(C401-Pad1)
- U602 pad 5: /Connector/MCU_SPI3_MOSI -> /MCU/MCU_SPI3_MOSI
- U602 pad 6: /Connector/MCU_SPI3_SCLK -> /MCU/MCU_SPI3_SCLK
- U603 pad 5: /Connector/MCU_SPI3_MOSI -> /MCU/MCU_SPI3_MOSI
- U603 pad 6: /Connector/MCU_SPI3_SCLK -> /MCU/MCU_SPI3_SCLK
- U604 pad 1: /Connector/FPGA2_SPI4_SLCK -> /Connector/RELAY2_SCLK
- U604 pad 10: /MCU/I2C_SDA -> /Connector/RELAY2_~CS3
- U604 pad 11: /MCU/I2C_SCL -> (no net)
- U604 pad 111: /Connector/MCU_SPI3_SCLK -> /MCU/MCU_SPI3_SCLK
- U604 pad 113: /Connector/MCU_SPI3_MOSI -> /MCU/MCU_SPI3_MOSI
- U604 pad 134: /FPGA/FPGA1_CDONE -> (no net)
- U604 pad 135: /FPGA/FPGA1_CRESET_B -> (no net)
- U604 pad 139: /FPGA/FPGA1_CBSEL0 -> (no net)
- U604 pad 140: /FPGA/FPGA1_CBSEL1 -> (no net)
- U604 pad 15: (no net) -> /MCU/RELAY1_~RST
- U604 pad 18: /FPGA/FPGA1_SPI5_CS -> (no net)
- U604 pad 19: /FPGA/FPGA1_SPI5_SLCK -> /MCU/RELAY1_SCLK
- U604 pad 2: (no net) -> /Connector/RELAY2_~RST
- U604 pad 20: /FPGA/FPGA1_SPI5_MISO -> /MCU/RELAY1_SO
- U604 pad 21: /FPGA/FPGA1_SPI5_MOSI -> /MCU/RELAY1_SI
- U604 pad 22: (no net) -> /MCU/RELAY1_~CS0
- U604 pad 3: /Connector/FPGA2_SPI4_CS -> (no net)
- U604 pad 32: /MCU/MCU_VREF+ -> /MCU/MCU_VDDA
- U604 pad 4: /Connector/FPGA2_SPI4_MISO -> /Connector/RELAY2_SO
- U604 pad 46: /Connector/MODULE_DETECT -> /Connector/MODULE_DETECT0
- U604 pad 47: (no net) -> /Connector/MODULE_DETECT1
- U604 pad 49: (no net) -> /MCU/RELAY1_~CS1
- U604 pad 5: /Connector/FPGA2_SPI4_MOSI -> /Connector/RELAY2_SI
- U604 pad 50: (no net) -> /MCU/RELAY1_~CS2
- U604 pad 53: (no net) -> /MCU/RELAY1_~CS3
- U604 pad 54: (no net) -> /MCU/I2C_SCL
- U604 pad 55: (no net) -> /MCU/I2C_SDA
- U604 pad 6: Net-(R309-Pad1) -> Net-(C607-Pad1)
- U604 pad 65: /Connector/FPGA2_CDONE -> (no net)
- U604 pad 66: /Connector/FPGA2_CRESET_B -> (no net)
- U604 pad 67: /Connector/FPGA2_CBSEL0 -> (no net)
- U604 pad 68: /Connector/FPGA2_CBSEL1 -> (no net)
- U604 pad 7: (no net) -> /Connector/RELAY2_~CS0
- U604 pad 8: (no net) -> /Connector/RELAY2_~CS1
- U604 pad 9: (no net) -> /Connector/RELAY2_~CS2
- U604 pad 96: /Connector/FPGA2_CFG_CS -> (no net)
- U604 pad 97: /FPGA/FPGA1_CFG_CS -> (no net)
Routing:
- net /Relays/RELAY9A: track 0.00 -> 47.0 mm, vias 0 -> 1
- net /Relays/RELAY10A: track 0.00 -> 42.2 mm, vias 0 -> 1
- net /Relays/RELAY11A: track 0.00 -> 37.5 mm, vias 0 -> 1
- net /Relays/RELAY12A: track 0.00 -> 32.7 mm, vias 0 -> 1
- net /Connector/F: track 0.00 -> 9.91 mm
- net /Connector/E: track 0.00 -> 9.91 mm
- net /Connector/D: track 0.00 -> 9.91 mm
- net /Connector/C: track 0.00 -> 9.91 mm
- net /Connector/B: track 0.00 -> 9.91 mm
- net /Connector/A: track 0.00 -> 9.91 mm
Other:
- outline, holes or cut-outs redrawn
- copper layers 2 -> 4
- net class Default: clearance 0.2 -> 0.127; trace_width 0.25 -> 0.127; via_dia 0.8 -> 0.5; via_drill 0.4 -> 0.2
- net class Relay signal 100V added: clearance 0.15, trace_width 0.381, via_dia 0.8, via_drill 0.4
- rule trace_clearance: 0.2 -> 0.127
- rule via_min_drill: 0.3 -> 0.2
- rule via_min_size: 0.4 -> 0.5
