File: hardware/project/ETH6C16MUX/Relays.sch (KiCad schematic (older format))
At the start: 182 parts

Commit message: Schematic design
Parts:
- removed K? (x120): HE3621A0500, symbol ETH6C16MUX:HE3621A0500
- added K601, K602, K603, K604, K605, K606, K607, K608, K609, K610, K611, K612, K613, K614, K615, K616, K617, K618, K619, K620, K621, K622, K623, K624, K625, K626, K627, K628, K629, K630, K631, K632, K633, K634, K635, K636, K637, K638, K639, K640, K641, K642, K643, K644, K645, K646, K647, K648, K649, K650, K651, K652, K653, K654: HE3621A0500, ETH6C16MXU:HE360_x-5331272-5, symbol ETH6C16MUX:HE3600
- D601, D602, D603, D604, D605, D606, D607, D608, D609, D610, D611, D612, D613, D614, D615, D616, D617, D618, D619, D620, D621, D622, D623, D624, D625, D626, D627, D628, D629, D630, D631, D632, D633, D634, D635, D636, D637, D638, D639, D640, D641, D642, D643, D644, D645, D646, D647, D648, D649, D650, D651, D652, D653, D654: renamed from D?; footprint (none) -> Diode_SMD:D_SOD-323_HandSoldering
- U601, U602, U603, U604, U605, U606, U607: renamed from U?; footprint (none) -> Package_SO:SOIC-18W_7.5x11.6mm_P1.27mm
- gave numbers to parts that had none: 1
Connections:
- net labels added: RELAY0, RELAY1, RELAY10, RELAY11, RELAY12, RELAY13, RELAY14, RELAY15, RELAY16, RELAY17, RELAY18, RELAY19, RELAY2, RELAY20, RELAY21, RELAY22, RELAY23, RELAY24, RELAY25, RELAY26, RELAY27, RELAY28, RELAY29, RELAY3, RELAY30, RELAY31, RELAY32, RELAY33, RELAY34, RELAY35, RELAY36, RELAY37, RELAY38, RELAY39, RELAY4, RELAY40, RELAY41, RELAY42, RELAY43, RELAY44, RELAY45, RELAY46, RELAY47, RELAY48, RELAY49, RELAY5, RELAY50, RELAY51, RELAY52, RELAY53, RELAY6, RELAY7, RELAY8, RELAY9, RELAY[0..53]
- net labels removed: CTRI_10A, CTRI_10B, CTRI_10C, CTRI_11A, CTRI_11B, CTRI_11C, CTRI_12A, CTRI_12B, CTRI_12C, CTRI_13A, CTRI_13B, CTRI_13C, CTRI_14A, CTRI_14B, CTRI_14C, CTRI_15A, CTRI_15B, CTRI_15C, CTRI_16A, CTRI_16B, CTRI_16C, CTRI_1A, CTRI_1B, CTRI_1C, CTRI_2A, CTRI_2B, CTRI_2C, CTRI_3A, CTRI_3B, CTRI_3C, CTRI_4A, CTRI_4B, CTRI_4C, CTRI_5A, CTRI_5B, CTRI_5C, CTRI_6A, CTRI_6B, CTRI_6C, CTRI_7A, CTRI_7B, CTRI_7C, CTRI_8A, CTRI_8B, CTRI_8C, CTRI_9A, CTRI_9B, CTRI_9C, CTRI_A, CTRI_B, CTRI_C, CTRI_D, CTRI_E, CTRI_F, RELAY_CTR
- wire segments 855 -> 819
Other:
- note added: "REED RELAYS AND CONNECTED"
- note removed: "REED RELAYS"
- moved on the sheet: U601, U602, U603, U604, U605, U606, U607

Commit message: PCB design, need to redesign of the board to board connectors.
Parts:
- removed D601, D602, D603, D604, D605, D606, D607, D608, D609, D610, D611, D612, D613, D614, D615, D616, D617, D618, D619, D620, D621, D622, D623, D624, D625, D626, D627, D628, D629, D630, D631, D632, D633, D634, D635, D636, D637, D638, D639, D640, D641, D642, D643, D644, D645, D646, D647, D648, D649, D650, D651, D652, D653, D654: 1N4148WS, Diode_SMD:D_SOD-323_HandSoldering, symbol Device:D
- J601: value D3408-5202-AR -> 1-103673-5; footprint (none) -> ETH6C16MXU:1-103673-5
Connections:
- net labels added: RELAY10A, RELAY10B, RELAY10C, RELAY11A, RELAY11B, RELAY11C, RELAY12A, RELAY12B, RELAY12C, RELAY13A, RELAY13B, RELAY13C, RELAY14A, RELAY14B, RELAY14C, RELAY15A, RELAY15B, RELAY15C, RELAY16A, RELAY16B, RELAY16C, RELAY1A, RELAY1B, RELAY1C, RELAY2A, RELAY2B, RELAY2C, RELAY3A, RELAY3B, RELAY3C, RELAY4A, RELAY4B, RELAY4C, RELAY5A, RELAY5B, RELAY5C, RELAY6A, RELAY6B, RELAY6C, RELAY7A, RELAY7B, RELAY7C, RELAY8A, RELAY8B, RELAY8C, RELAY9A, RELAY9B, RELAY9C, RELAYA, RELAYB, RELAYC, RELAYD, RELAYE, RELAYF
- net labels removed: CTRO_10A, CTRO_10B, CTRO_10C, CTRO_11A, CTRO_11B, CTRO_11C, CTRO_12A, CTRO_12B, CTRO_12C, CTRO_13A, CTRO_13B, CTRO_13C, CTRO_14A, CTRO_14B, CTRO_14C, CTRO_15A, CTRO_15B, CTRO_15C, CTRO_16A, CTRO_16B, CTRO_16C, CTRO_1A, CTRO_1B, CTRO_1C, CTRO_2A, CTRO_2B, CTRO_2C, CTRO_3A, CTRO_3B, CTRO_3C, CTRO_4A, CTRO_4B, CTRO_4C, CTRO_5A, CTRO_5B, CTRO_5C, CTRO_6A, CTRO_6B, CTRO_6C, CTRO_7A, CTRO_7B, CTRO_7C, CTRO_8A, CTRO_8B, CTRO_8C, CTRO_9A, CTRO_9B, CTRO_9C, CTRO_A, CTRO_B, CTRO_C, CTRO_D, CTRO_E, CTRO_F
- wire segments 819 -> 549
Other:
- note added: "1-487526-5 \n\n1-104480-6\n104479-9 \n1-104480-2 \n104480-2"
- note removed: "D3408-5302-AR"
- moved on the sheet: K601B, K602B, K603B, K604B, K605B, K606B, K607B, K608B, K609B, K610B, K611B, K612B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

Commit message: PCB layout, deleted USB.
Parts:
- removed J601: 1-103673-5, ETH6C16MXU:1-103673-5, symbol Connector_Generic:Conn_01x16
- added J501: Conn_02x08_Counter_Clockwise, Connector_IDC:IDC-Header_2x08_P2.54mm_Horizontal_Lock, symbol Connector_Generic:Conn_02x08_Counter_Clockwise
- renumbered K601 to K501, K602 to K502, K603 to K503, K604 to K504, K605 to K505, K606 to K506, K607 to K507, K608 to K508, K609 to K509, K610 to K510, K611 to K511, K612 to K512, K613 to K513, K614 to K514, K615 to K515, K616 to K516, K617 to K517, K618 to K518, K619 to K519, K620 to K520, K621 to K521, K622 to K522, K623 to K523, K624 to K524, K625 to K525, K626 to K526, K627 to K527, K628 to K528, K629 to K529, K630 to K530, K631 to K531, K632 to K532, K633 to K533, K634 to K534, K635 to K535, K636 to K536, K637 to K537, K638 to K538, K639 to K539, K640 to K540, K641 to K541, K642 to K542, K643 to K543, K644 to K544, K645 to K545, K646 to K546, K647 to K547, K648 to K548, K649 to K549, K650 to K550, K651 to K551, K652 to K552, K653 to K553, K654 to K554, U601 to U501, U602 to U502, U603 to U503, U604 to U504, U605 to U505, U606 to U506, U607 to U507
Connections:
- net PIN1: now also J501.1 (Pin_1)
- net PIN10: now also J501.10 (Pin_10)
- net PIN11: now also J501.11 (Pin_11)
- net PIN12: now also J501.12 (Pin_12)
- net PIN13: now also J501.13 (Pin_13)
- net PIN14: now also J501.14 (Pin_14)
- net PIN15: now also J501.15 (Pin_15)
- net PIN16: now also J501.16 (Pin_16)
- net PIN2: now also J501.2 (Pin_2)
- net PIN3: now also J501.3 (Pin_3)
- net PIN4: now also J501.4 (Pin_4)
- net PIN5: now also J501.5 (Pin_5)
- net PIN6: now also J501.6 (Pin_6)
- net PIN7: now also J501.7 (Pin_7)
- net PIN8: now also J501.8 (Pin_8)
- net PIN9: now also J501.9 (Pin_9)

Commit message: Deleted FPGA part and change it for SPI IO chips. Change power supply circuit.
Parts:
- removed U501, U502, U503, U504, U505, U506, U507: ULN2803A, Package_SO:SOIC-18W_7.5x11.6mm_P1.27mm, symbol Transistor_Array:ULN2803A
- added U301, U302, U303, U304: MCZ33996, ETH6C16MXU:HSOP-32-1EP_7.5x11.0mm_P0.65mm_ThermalVias, symbol ETH6C16MUX:MCZ33996
- renumbered J501 to J301, K501 to K301, K502 to K302, K503 to K303, K504 to K304, K505 to K305, K506 to K306, K507 to K307, K508 to K308, K509 to K309, K510 to K310, K511 to K311, K512 to K312, K513 to K313, K514 to K314, K515 to K315, K516 to K316, K517 to K317, K518 to K318, K519 to K319, K520 to K320, K521 to K321, K522 to K322, K523 to K323, K524 to K324, K525 to K325, K526 to K326, K527 to K327, K528 to K328, K529 to K329, K530 to K330, K531 to K331, K532 to K332, K533 to K333, K534 to K334, K535 to K335, K536 to K336, K537 to K337, K538 to K338, K539 to K339, K540 to K340, K541 to K341, K542 to K342, K543 to K343, K544 to K344, K545 to K345, K546 to K346, K547 to K347, K548 to K348, K549 to K349, K550 to K350, K551 to K351, K552 to K352, K553 to K353, K554 to K354
Connections:
- net +5V: now also U301.6 (VPWR), U302.6 (VPWR), U303.6 (VPWR), U304.6 (VPWR)
- net GND: now also U301.10 (GND), U301.23 (GND), U301.24 (GND), U301.25 (GND), U301.26 (GND), U301.33 (EP), U301.7 (GND), U301.8 (GND), U301.9 (GND), U302.10 (GND), U302.23 (GND), U302.24 (GND), U302.25 (GND), U302.26 (GND), U302.33 (EP), U302.7 (GND), U302.8 (GND), U302.9 (GND), U303.10 (GND), U303.23 (GND), U303.24 (GND), U303.25 (GND), U303.26 (GND), U303.33 (EP), U303.7 (GND), U303.8 (GND), U303.9 (GND), U304.10 (GND), U304.23 (GND), U304.24 (GND), U304.25 (GND), U304.26 (GND), U304.33 (EP), U304.7 (GND), U304.8 (GND), U304.9 (GND)
- net RELAY10A: now also U301.18 (OUT9)
- net RELAY10B: now also U303.18 (OUT9)
- net RELAY10C: now also U302.18 (OUT9)
- net RELAY11A: now also U301.20 (OUT10)
- net RELAY11B: now also U303.20 (OUT10)
- net RELAY11C: now also U302.20 (OUT10)
- net RELAY12A: now also U301.21 (OUT11)
- net RELAY12B: now also U303.21 (OUT11)
- net RELAY12C: now also U302.21 (OUT11)
- net RELAY13A: now also U301.28 (OUT12)
- net RELAY13B: now also U303.28 (OUT12)
- net RELAY13C: now also U302.28 (OUT12)
- net RELAY14A: now also U301.29 (OUT13)
- net RELAY14B: now also U303.29 (OUT13)
- net RELAY14C: now also U302.29 (OUT13)
- net RELAY15A: now also U301.31 (OUT14)
- net RELAY15B: now also U303.31 (OUT14)
- net RELAY15C: now also U302.31 (OUT14)
- net RELAY16A: now also U301.32 (OUT15)
- net RELAY16B: now also U303.32 (OUT15)
- net RELAY16C: now also U302.32 (OUT15)
- net RELAY1A: now also U301.1 (OUT0)
- net RELAY1B: now also U303.1 (OUT0)
- net RELAY1C: now also U302.1 (OUT0)
- net RELAY2A: now also U301.2 (OUT1)
- net RELAY2B: now also U303.2 (OUT1)
- net RELAY2C: now also U302.2 (OUT1)
- net RELAY3A: now also U301.4 (OUT2)
- net RELAY3B: now also U303.4 (OUT2)
- net RELAY3C: now also U302.4 (OUT2)
- net RELAY4A: now also U301.5 (OUT3)
- net RELAY4B: now also U303.5 (OUT3)
- net RELAY4C: now also U302.5 (OUT3)
- net RELAY5A: now also U301.12 (OUT4)
- net RELAY5B: now also U303.12 (OUT4)
- net RELAY5C: now also U302.12 (OUT4)
- net RELAY6A: now also U301.13 (OUT5)
- net RELAY6B: now also U303.13 (OUT5)
- net RELAY6C: now also U302.13 (OUT5)
- net RELAY7A: now also U301.15 (OUT6)
- net RELAY7B: now also U303.15 (OUT6)
- net RELAY7C: now also U302.15 (OUT6)
- net RELAY8A: now also U301.16 (OUT7)
- net RELAY8B: now also U303.16 (OUT7)
- net RELAY8C: now also U302.16 (OUT7)
- net RELAY9A: now also U301.17 (OUT8)
- net RELAY9B: now also U303.17 (OUT8)
- net RELAY9C: now also U302.17 (OUT8)
- net RELAYA: now also U304.1 (OUT0)
- net RELAYB: now also U304.2 (OUT1)
- net RELAYC: now also U304.4 (OUT2)
- net RELAYD: now also U304.5 (OUT3)
- net RELAYE: now also U304.12 (OUT4)
- net RELAYF: now also U304.13 (OUT5)
- new net +3V3: U301.3 (SOPWR), U302.3 (SOPWR), U303.3 (SOPWR), U304.3 (SOPWR)
- new net RELAY1_SCLK: U301.11 (SCLK), U302.11 (SCLK), U303.11 (SCLK), U304.11 (SCLK)
- new net RELAY1_SI: U301.19 (SI), U302.19 (SI), U303.19 (SI), U304.19 (SI)
- new net RELAY1_SO: U301.22 (SO), U302.22 (SO), U303.22 (SO), U304.22 (SO)
- new net RELAY1_~CS0: U301.14 (~CS)
- new net RELAY1_~CS1: U303.14 (~CS)
- new net RELAY1_~CS2: U302.14 (~CS)
- new net RELAY1_~CS3: U304.14 (~CS)
- new net RELAY1_~RST: U301.27 (~RST), U302.27 (~RST), U303.27 (~RST), U304.27 (~RST)
- no-connect marks 4 -> 14
