File: hardware/project/ETH6C20MUX/ETH6C20MUX.sch (KiCad schematic (older format))
At the start: 3 parts, among them M101 60817-096

Commit message: Ranamed project to ETH6C20MUX. Added 4 channels. Schematic redesign and PCB layout.
Parts:
- removed M101: 60817-096, ETH6C16MXU:60817-096, symbol ETH6C16MUX:60817-096
Connections:
- wire segments 39 -> 40
Changed lines of the file:
@@
 F4 "RX+" B R 7900 4400 50
 F5 "RX-" B R 7900 4500 50
-F6 "ETH_RMII_TX1" B L 6700 4100 50
-F7 "ETH_RMII_TX0" B L 6700 4200 50
-F8 "ETH_RMII_TXEN" B L 6700 4300 50
-F9 "ETH_RMII_RX0" B L 6700 4400 50
-F10 "ETH_RMII_RX1" B L 6700 4500 50
-F11 "ETH_RMII_CRS_DV" B L 6700 4600 50
-F12 "ETH_RMII_MDIO" B L 6700 4700 50
-F13 "ETH_RMII_MDC" B L 6700 4800 50
-F14 "ETH_~RST" B L 6700 4900 50
-F15 "ETH_~INT" B L 6700 5000 50
-F16 "ETH_RMII_REF_CLK" O L 6700 5100 50
+F6 "RMII_TXD1" B L 6700 4100 50
+F7 "RMII_TXD0" B L 6700 4200 50
+F8 "RMII_TXEN" B L 6700 4300 50
+F9 "RMII_RXD0" B L 6700 4400 50
+F10 "RMII_RXD1" B L 6700 4500 50
+F11 "RMII_CRS_DV" B L 6700 4600 50
+F12 "RMII_MDIO" B L 6700 4700 50
+F13 "RMII_MDC" B L 6700 4800 50
+F14 "NRST" B L 6700 4900 50
+F15 "REF_CLK" B L 6700 5000 50
 $EndSheet
 $Sheet
@@
 F10 "RELAY1_~CS2" I R 3650 1950 50
 F11 "RELAY1_~CS3" I R 3650 2050 50
-F12 "RELAY1_SCLK" I R 3650 2150 50
-F13 "RELAY1_SI" I R 3650 2250 50
-F14 "RELAY1_SO" O R 3650 2350 50
-F15 "RELAY1_~RST" I R 3650 2450 50
+F12 "RELAY1_SCLK" I R 3650 2250 50
+F13 "RELAY1_SI" I R 3650 2350 50
+F14 "RELAY1_SO" O R 3650 2450 50
+F15 "RELAY1_~RST" I R 3650 2550 50
+F16 "RELAY1_~CS4" I R 3650 2150 50
 $EndSheet
 Text Notes 950  7300 0    50   ~ 0
@@
 $EndSheet
 Wire Wire Line
-	6400 5100 6700 5100
-Wire Wire Line
-	6700 5000 6400 5000
+	6400 5000 6700 5000
 Wire Wire Line
 	6400 4900 6700 4900
@@
 F13 "RELAY2_~CS1" I L 8200 1850 50
 F14 "RELAY2_~CS0" I L 8200 1750 50
-F15 "RELAY2_SCLK" I L 8200 2150 50
-F16 "RELAY2_SI" I L 8200 2250 50
-F17 "RELAY2_SO" O L 8200 2350 50
-F18 "RELAY2_~RST" O L 8200 2450 50
-F19 "MODULE_DETECT0" I L 8200 2550 50
-F20 "MODULE_DETECT1" I L 8200 2650 50
+F15 "RELAY2_SCLK" I L 8200 2250 50
+F16 "RELAY2_SI" I L 8200 2350 50
+F17 "RELAY2_SO" O L 8200 2450 50
+F18 "RELAY2_~RST" O L 8200 2550 50
+F19 "MODULE_DETECT0" I L 8200 2650 50
+F20 "MODULE_DETECT1" I L 8200 2750 50
 F21 "RELAY2_~CS3" I L 8200 2050 50
+F22 "RELAY2_~CS4" I L 8200 2150 50
 $EndSheet
 Wire Wire Line
@@
 Wire Wire Line
 	6400 2550 8200 2550
+Wire Wire Line
+	6400 2650 8200 2650
 $Sheet
 S 4500 1650 1900 3550
@@
 F0 "MCU" 50
 F1 "MCU.sch" 50
-F2 "ETH_RMII_REF_CLK" I R 6400 5100 50
-F3 "ETH_~INT" B R 6400 5000 50
-F4 "ETH_~RST" B R 6400 4900 50
-F5 "ETH_RMII_MDC" B R 6400 4800 50
-F6 "ETH_RMII_MDIO" B R 6400 4700 50
-F7 "ETH_RMII_CRS_DV" B R 6400 4600 50
-F8 "ETH_RMII_RX1" B R 6400 4500 50
-F9 "ETH_RMII_RX0" B R 6400 4400 50
-F10 "ETH_RMII_TXEN" B R 6400 4300 50
-F11 "ETH_RMII_TX0" B R 6400 4200 50
-F12 "ETH_RMII_TX1" B R 6400 4100 50
-F13 "RELAY1_SCLK" O L 4500 2150 50
-F14 "RELAY1_SI" O L 4500 2250 50
-F15 "RELAY1_SO" I L 4500 2350 50
-F16 "RELAY1_~RST" I L 4500 2450 50
-F17 "RELAY1_~CS3" O L 4500 2050 50
-F18 "RELAY1_~CS2" O L 4500 1950 50
-F19 "RELAY1_~CS1" O L 4500 1850 50
-F20 "RELAY1_~CS0" O L 4500 1750 50
-F21 "RELAY2_SCLK" O R 6400 2150 50
-F22 "RELAY2_SI" O R 6400 2250 50
-F23 "RELAY2_SO" I R 6400 2350 50
-F24 "RELAY2_~RST" I R 6400 2450 50
-F25 "RELAY2_~CS3" O R 6400 2050 50
-F26 "RELAY2_~CS2" O R 6400 1950 50
-F27 "RELAY2_~CS1" O R 6400 1850 50
-F28 "RELAY2_~CS0" O R 6400 1750 50
-F29 "MODULE_DETECT0" O R 6400 2550 50
-F30 "MODULE_DETECT1" O R 6400 2650 50
-$EndSheet
-Wire Wire Line
-	6400 2650 8200 2650
-$Comp
-L ETH6C16MUX:60817-096 M101
-U 1 1 5D83A8D3
-P 4650 7050
-F 0 "M101" H 4978 7396 50  0000 L CNN
-F 1 "60817-096" H 4978 7305 50  0000 L CNN
-F 2 "ETH6C16MXU:60817-096" H 4650 7050 50  0001 C CNN
-F 3 "" H 4650 7050 50  0001 C CNN
-	1    4650 7050
-	1    0    0    -1
-$EndComp
+F2 "RELAY1_SCLK" O L 4500 2250 50
+F3 "RELAY1_SI" O L 4500 2350 50
+F4 "RELAY1_SO" I L 4500 2450 50
+F5 "RELAY1_~RST" I L 4500 2550 50
+F6 "RELAY1_~CS3" O L 4500 2050 50
+F7 "RELAY1_~CS2" O L 4500 1950 50
+F8 "RELAY1_~CS1" O L 4500 1850 50
+F9 "RELAY1_~CS0" O L 4500 1750 50
+F10 "RELAY2_SCLK" O R 6400 2250 50
+F11 "RELAY2_SI" O R 6400 2350 50
+F12 "RELAY2_SO" I R 6400 2450 50
+F13 "RELAY2_~RST" I R 6400 2550 50
+F14 "RELAY2_~CS3" O R 6400 2050 50
+F15 "RELAY2_~CS2" O R 6400 1950 50
+F16 "RELAY2_~CS1" O R 6400 1850 50
+F17 "RELAY2_~CS0" O R 6400 1750 50
+F18 "MODULE_DETECT0" O R 6400 2650 50
+F19 "MODULE_DETECT1" O R 6400 2750 50
+F20 "RMII_REF_CLK" I R 6400 5000 50
+F21 "NRST" B R 6400 4900 50
+F22 "RMII_MDC" B R 6400 4800 50
+F23 "RMII_CRS_DV" B R 6400 4600 50
+F24 "RMII_RXD1" B R 6400 4500 50
+F25 "RMII_RXD0" B R 6400 4400 50
+F26 "RMII_MDIO" B R 6400 4700 50
+F27 "RELAY1_~CS4" O L 4500 2150 50
+F28 "RELAY2_~CS4" O R 6400 2150 50
+F29 "RMII_TXEN" B R 6400 4300 50
+F30 "RMII_TX0" B R 6400 4200 50
+F31 "RMII_TX1" B R 6400 4100 50
+$EndSheet
+Wire Wire Line
+	3650 2550 4500 2550
+Wire Wire Line
+	8200 2750 6400 2750
 $EndSCHEMATC
