File: hardware/project/ETH6C20MUX/ETH6C20MUX.sch (KiCad schematic (older format))
At the start: 2 parts

Commit message: PCB redesign
Parts:
- added H103: MountingHole, MountingHole:MountingHole_2.7mm_M2.5_DIN965_Pad, symbol Mechanical:MountingHole
- H101, H102: footprint MountingHole:MountingHole_3.2mm_M3_DIN965_Pad -> MountingHole:MountingHole_2.7mm_M2.5_DIN965_Pad
Changed lines of the file:
@@
 F 0 "H101" H 3050 6946 50  0000 L CNN
 F 1 "MountingHole" H 3050 6855 50  0000 L CNN
-F 2 "MountingHole:MountingHole_3.2mm_M3_DIN965_Pad" H 2950 6900 50  0001 C CNN
+F 2 "MountingHole:MountingHole_2.7mm_M2.5_DIN965_Pad" H 2950 6900 50  0001 C CNN
 F 3 "~" H 2950 6900 50  0001 C CNN
 	1    2950 6900
@@
 F 0 "H102" H 4000 6946 50  0000 L CNN
 F 1 "MountingHole" H 4000 6855 50  0000 L CNN
-F 2 "MountingHole:MountingHole_3.2mm_M3_DIN965_Pad" H 3900 6900 50  0001 C CNN
+F 2 "MountingHole:MountingHole_2.7mm_M2.5_DIN965_Pad" H 3900 6900 50  0001 C CNN
 F 3 "~" H 3900 6900 50  0001 C CNN
 	1    3900 6900
@@
 Wire Wire Line
 	8200 2750 6400 2750
+$Comp
+L Mechanical:MountingHole H103
+U 1 1 60B19546
+P 4800 6900
+F 0 "H103" H 4900 6946 50  0000 L CNN
+F 1 "MountingHole" H 4900 6855 50  0000 L CNN
+F 2 "MountingHole:MountingHole_2.7mm_M2.5_DIN965_Pad" H 4800 6900 50  0001 C CNN
+F 3 "~" H 4800 6900 50  0001 C CNN
+	1    4800 6900
+	1    0    0    -1
+$EndComp
 $EndSCHEMATC
