File: hardware/project/ETH6C20MUX/MCU.sch (KiCad schematic (older format))
At the start: 42 parts, among them J601 Conn_02x05, J602 Conn_02x01, J603 Conn_02x01, U601 ASDM1-20.000MHZ-LC-T, U602 S25FL064L_SOIC, U603 S25FL064L_SOIC, U604 STM32F765ZGT6, U605 MCP9804

Commit message: Ranamed project to ETH6C20MUX. Added 4 channels. Schematic redesign and PCB layout.
Parts:
- removed D601: 150121M153000, ETH6C16MXU:150121M153000, symbol Device:LED_ARGB
- removed J602: Conn_02x01, Connector_PinHeader_2.54mm:PinHeader_1x02_P2.54mm_Vertical, symbol Connector_Generic:Conn_02x01
- removed R601: 220, Resistor_SMD:R_0603_1608Metric_Pad1.05x0.95mm_HandSolder, symbol Device:R
- removed R603, R604: 4k7, Resistor_SMD:R_0603_1608Metric_Pad1.05x0.95mm_HandSolder, symbol Device:R
- removed R606: 523, Resistor_SMD:R_0603_1608Metric_Pad1.05x0.95mm_HandSolder, symbol Device:R
- removed R607, R608: 330, Resistor_SMD:R_0603_1608Metric_Pad1.05x0.95mm_HandSolder, symbol Device:R
- removed R609: 0, Resistor_SMD:R_0603_1608Metric_Pad1.05x0.95mm_HandSolder, symbol Device:R
- removed R611: 10k, Resistor_SMD:R_0603_1608Metric_Pad1.05x0.95mm_HandSolder, symbol Device:R
- removed U601: ASDM1-20.000MHZ-LC-T, Oscillator:Oscillator_SMD_Abracon_ASDMB-4Pin_2.5x2.0mm, symbol Oscillator:ASDMB-xxxMHz
- removed U605: MCP9804, Package_SO:MSOP-8_3x3mm_P0.65mm, symbol Sensor_Temperature:MCP9804_MSOP
- added C602: 8p, Capacitor_SMD:C_0603_1608Metric_Pad1.05x0.95mm_HandSolder, symbol Device:C
- added Y601: NX3225GD-8MHZ-STD-CRA-3, ETH6C16MXU:NX3225GD, symbol Device:Crystal
- C601: value 100n -> 8p
- R608: renamed from R610; value R -> 10k
- U601: renamed from U602; symbol ETH6C16MUX:S25FL064L_SOIC -> ETH6C20MUX:S25FL064L_SOIC
- U602: renamed from U603; symbol ETH6C16MUX:S25FL064L_SOIC -> ETH6C20MUX:S25FL064L_SOIC
- U603: renamed from U604; footprint Package_QFP:TQFP-144_20x20mm_P0.5mm -> ETH6C16MXU:TQFP-144_20x20mm_P0.5mm; symbol ETH6C16MUX:STM32F765ZGT6 -> ETH6C20MUX:STM32F765ZGT6
- renumbered C602 to C603, C603 to C604, C604 to C605, C605 to C606, C606 to C607, C607 to C608, C608 to C609, C609 to C610, C610 to C611, C611 to C612, C612 to C613, C613 to C614, C614 to C615, C615 to C616, C616 to C617, C617 to C618, C618 to C619, C619 to C620, C620 to C621, J603 to J602, R602 to R601, R605 to R604, R612 to R609
Connections:
- net labels added: NRST, RELAY1_~CS4, RELAY2_~CS4, RMII_CRS_DV, RMII_MDC, RMII_MDIO, RMII_REF_CLK, RMII_RXD0, RMII_RXD1, RMII_TX0, RMII_TX1, RMII_TXEN
- net labels removed: ETH_RMII_CRS_DV, ETH_RMII_MDC, ETH_RMII_MDIO, ETH_RMII_REF_CLK, ETH_RMII_RX0, ETH_RMII_RX1, ETH_RMII_TX0, ETH_RMII_TX1, ETH_RMII_TXEN, ETH_~INT, ETH_~RST, I2C_SCL, I2C_SDA, LED_BLUE, LED_GREEN, LED_RED, MCU_BOOT
- wire segments 253 -> 220
- no-connect marks 72 -> 74
Other:
- moved on the sheet: J602, R609
