File: hardware/project/ETH6C20MUX/MCU.sch (KiCad schematic (older format))
At the start: 32 parts, among them J601 Conn_02x05, J602 Conn_02x01, U601 S25FL064L_SOIC, U602 S25FL064L_SOIC, U603 STM32F765ZGT6, Y601 NX3225GD-8MHZ-STD-CRA-3

Commit message: Updated PCB. Added 3D components. Started BOM list.
Parts:
- U603: footprint ETH6C16MXU:TQFP-144_20x20mm_P0.5mm -> ETH6C20MUX:TQFP-144_20x20mm_P0.5mm
- Y601: footprint ETH6C16MXU:NX3225GD -> ETH6C20MUX:NX3225GD
Changed lines of the file:
@@
 F 0 "Y601" V 2254 1681 50  0000 L CNN
 F 1 "NX3225GD-8MHZ-STD-CRA-3" V 2345 1681 50  0000 L CNN
-F 2 "ETH6C16MXU:NX3225GD" H 2300 1550 50  0001 C CNN
+F 2 "ETH6C20MUX:NX3225GD" H 2300 1550 50  0001 C CNN
 F 3 "~" H 2300 1550 50  0001 C CNN
 	1    2300 1550
@@
 F 0 "U603" H 4100 9150 50  0000 C CNN
 F 1 "STM32F765ZGT6" H 14650 9150 50  0000 C CNN
-F 2 "ETH6C16MXU:TQFP-144_20x20mm_P0.5mm" H 25350 6750 50  0001 C CNN
+F 2 "ETH6C20MUX:TQFP-144_20x20mm_P0.5mm" H 25350 6750 50  0001 C CNN
 F 3 "" H 25350 6750 50  0001 C CNN
 	1    9450 5250
