File: hardware/project/ETH6C20MUX/Relays.sch (KiCad schematic (older format))
At the start: 72 parts, among them J301 Conn_02x10_Counter_Clockwise, K301 HE3621A0500, K302 HE3621A0500, K303 HE3621A0500, K304 HE3621A0500, K305 HE3621A0500, K306 HE3621A0500, K307 HE3621A0500, K308 HE3621A0500, K309 HE3621A0500, K310 HE3621A0500, K311 HE3621A0500, K312 HE3621A0500, K313 HE3621A0500, K314 HE3621A0500, K315 HE3621A0500, K316 HE3621A0500, K317 HE3621A0500, K318 HE3621A0500, K319 HE3621A0500, K320 HE3621A0500, K321 HE3621A0500, K322 HE3621A0500, K323 HE3621A0500, K324 HE3621A0500, K325 HE3621A0500, K326 HE3621A0500, K327 HE3621A0500, K328 HE3621A0500, K329 HE3621A0500, K330 HE3621A0500, K331 HE3621A0500, K332 HE3621A0500, K333 HE3621A0500, K334 HE3621A0500, K335 HE3621A0500, K336 HE3621A0500, K337 HE3621A0500, K338 HE3621A0500, K339 HE3621A0500, K340 HE3621A0500, K341 HE3621A0500, K342 HE3621A0500, K343 HE3621A0500, K344 HE3621A0500, K345 HE3621A0500, K346 HE3621A0500, K347 HE3621A0500, K348 HE3621A0500, K349 HE3621A0500, K350 HE3621A0500, K351 HE3621A0500, K352 HE3621A0500, K353 HE3621A0500, K354 HE3621A0500, K355 HE3621A0500, K356 HE3621A0500, K357 HE3621A0500, K358 HE3621A0500, K359 HE3621A0500, K360 HE3621A0500, K361 HE3621A0500, K362 HE3621A0500, K363 HE3621A0500, K364 HE3621A0500, K365 HE3621A0500, K366 HE3621A0500, U301 MCZ33996, U302 MCZ33996, U303 MCZ33996, U304 MCZ33996, U305 MCZ33996

Commit message: Updated PCB. Added 3D components. Started BOM list.
Parts:
- added C301, C302, C303, C304, C305, C306, C307, C308, C309, C310: 100n, Capacitor_SMD:C_0603_1608Metric_Pad1.05x0.95mm_HandSolder, symbol Device:C
- J301: value Conn_02x10_Counter_Clockwise -> 5499141-4
- K301, K302, K303, K304, K305, K306, K307, K308, K309, K310, K311, K312, K313, K314, K315, K316, K317, K318, K319, K320, K321, K322, K323, K324, K325, K326, K327, K328, K329, K330, K331, K332, K333, K334, K335, K336, K337, K338, K339, K340, K341, K342, K343, K344, K345, K346, K347, K348, K349, K350, K351, K352, K353, K354, K355, K356, K357, K358, K359, K360, K361, K362, K363, K364, K365, K366: value HE3621A0500 -> HE3621A0510; footprint ETH6C16MXU:HE360_x-5331272-5 -> ETH6C20MUX:HE360_x-5331272-5
- U301, U302, U303, U304, U305: footprint ETH6C16MXU:HSOP-32-1EP_7.5x11.0mm_P0.65mm_ThermalVias -> ETH6C20MUX:HSOP-32-1EP_7.5x11.0mm_P0.65mm_ThermalVias
Connections:
- net +3V3: now also C301.1, C302.1, C303.1, C304.1, C305.1
- net +5V: now also C306.1, C307.1, C308.1, C309.1, C310.1
- net GND: now also C301.2, C302.2, C303.2, C304.2, C305.2, C306.2, C307.2, C308.2, C309.2, C310.2
Other:
- note removed: "1-487526-5 \n\n1-104480-6\n104479-9 \n1-104480-2 \n104480-2"
