File: hardware/project/ETH6C20MUX/Relays.sch (KiCad schematic (older format))
At the start: 82 parts, among them J301 5499141-4, K301 HE3621A0510, K302 HE3621A0510, K303 HE3621A0510, K304 HE3621A0510, K305 HE3621A0510, K306 HE3621A0510, K307 HE3621A0510, K308 HE3621A0510, K309 HE3621A0510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

Commit message: Small updates in PCB design.
Parts:
- K301, K302, K303, K304, K305, K306, K307, K308, K309, K310, K311, K312, K313, K314, K315, K316, K317, K318, K319, K320, K321, K322, K323, K324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: footprint ETH6C20MUX:HE360_x-5331272-5 -> ETH6C20MUX:HE360_x-5050462-8
