File: hardware/project/ETH6C20MUX/Power.sch (KiCad schematic (older format))
At the start: 16 parts, among them Q401 IRFR5410, U401 TSR2-2450, U402 MAX5902, U403 LM1117MPX-3.3

Commit message: Ranamed project to ETH6C20MUX. Added 4 channels. Schematic redesign and PCB layout.
Parts:
- U401: symbol ETH6C16MUX:TSR2-2450 -> ETH6C20MUX:TSR2-2450
- U402: symbol ETH6C16MUX:MAX5902 -> ETH6C20MUX:MAX5902
Changed lines of the file:
@@
 EESchema Schematic File Version 4
-LIBS:ETH6C16MUX-cache
+LIBS:ETH6C20MUX-cache
 EELAYER 30 0
 EELAYER END
@@
 $EndComp
 $Comp
-L power:GND #PWR0411
+L power:GND #PWR0410
 U 1 1 5D9353CB
 P 1350 7150
-F 0 "#PWR0411" H 1350 6900 50  0001 C CNN
+F 0 "#PWR0410" H 1350 6900 50  0001 C CNN
 F 1 "GND" H 1355 6977 50  0000 C CNN
 F 2 "" H 1350 7150 50  0001 C CNN
@@
 	1350 7150 1350 7000
 $Comp
-L power:+5V #PWR0410
+L power:+5V #PWR0409
 U 1 1 5D9B1EAC
 P 1750 7000
-F 0 "#PWR0410" H 1750 6850 50  0001 C CNN
+F 0 "#PWR0409" H 1750 6850 50  0001 C CNN
 F 1 "+5V" H 1765 7173 50  0000 C CNN
 F 2 "" H 1750 7000 50  0001 C CNN
@@
 $EndComp
 $Comp
-L power:PWR_FLAG #FLG0405
+L power:PWR_FLAG #FLG0404
 U 1 1 5D9B2CC2
 P 1750 7150
-F 0 "#FLG0405" H 1750 7225 50  0001 C CNN
+F 0 "#FLG0404" H 1750 7225 50  0001 C CNN
 F 1 "PWR_FLAG" H 1750 7323 50  0000 C CNN
 F 2 "" H 1750 7150 50  0001 C CNN
@@
 $EndComp
 $Comp
-L ETH6C16MUX:MAX5902 U402
+L ETH6C20MUX:MAX5902 U402
 U 1 1 5D6EBA14
 P 4800 1850
@@
 $EndComp
 $Comp
-L power:Earth #PWR0412
+L power:Earth #PWR0411
 U 1 1 5DA19730
 P 2250 7150
-F 0 "#PWR0412" H 2250 6900 50  0001 C CNN
+F 0 "#PWR0411" H 2250 6900 50  0001 C CNN
 F 1 "Earth" H 2250 7000 50  0001 C CNN
 F 2 "" H 2250 7150 50  0001 C CNN
@@
 Connection ~ 5900 2400
 $Comp
-L ETH6C16MUX:TSR2-2450 U401
+L ETH6C20MUX:TSR2-2450 U401
 U 1 1 5D7D1038
 P 8200 1450

Commit message: Updated PCB. Added 3D components. Started BOM list.
Parts:
- D402: footprint ETH6C16MXU:DO_214AA_REV -> ETH6C20MUX:DO_214AA_REV
- F401: footprint ETH6C16MXU:Fuse_SMD2920 -> ETH6C20MUX:Fuse_SMD2920
- Q401: footprint ETH6C16MXU:TO-252-2_Rectifier -> ETH6C20MUX:TO-252-2_Rectifier
- U401: footprint ETH6C16MXU:TSR2 -> ETH6C20MUX:TSR2
Changed lines of the file:
@@
 F 0 "D402" V 3204 1929 50  0000 L CNN
 F 1 "SM6T30AY" V 3295 1929 50  0000 L CNN
-F 2 "ETH6C16MXU:DO_214AA_REV" H 3250 1850 50  0001 C CNN
+F 2 "ETH6C20MUX:DO_214AA_REV" H 3250 1850 50  0001 C CNN
 F 3 "~" H 3250 1850 50  0001 C CNN
 	1    3250 1850
@@
 F 0 "Q401" V 5793 1450 50  0000 C CNN
 F 1 "IRFR5410" V 5702 1450 50  0000 C CNN
-F 2 "ETH6C16MXU:TO-252-2_Rectifier" H 5650 1550 50  0001 C CNN
+F 2 "ETH6C20MUX:TO-252-2_Rectifier" H 5650 1550 50  0001 C CNN
 F 3 "~" H 5450 1450 50  0001 C CNN
 	1    5450 1450
@@
 F 0 "F401" V 2803 1350 50  0000 C CNN
 F 1 "MF-LSMF185/33X" V 2894 1350 50  0000 C CNN
-F 2 "ETH6C16MXU:Fuse_SMD2920" V 2930 1350 50  0001 C CNN
+F 2 "ETH6C20MUX:Fuse_SMD2920" V 2930 1350 50  0001 C CNN
 F 3 "~" H 3000 1350 50  0001 C CNN
 	1    3000 1350
@@
 F 0 "U401" H 8200 1815 50  0000 C CNN
 F 1 "TSR2-2450" H 8200 1724 50  0000 C CNN
-F 2 "ETH6C16MXU:TSR2" H 8200 1750 50  0001 C CNN
+F 2 "ETH6C20MUX:TSR2" H 8200 1750 50  0001 C CNN
 F 3 "" H 8200 1750 50  0001 C CNN
 	1    8200 1450

Commit message: PCB redesign
Parts:
- C402, C405: footprint Capacitor_SMD:C_0603_1608Metric_Pad1.05x0.95mm_HandSolder -> Capacitor_SMD:C_0603_1608Metric_Pad1.08x0.95mm_HandSolder
- R401, R403: footprint Resistor_SMD:R_0603_1608Metric_Pad1.05x0.95mm_HandSolder -> Resistor_SMD:R_0603_1608Metric_Pad0.98x0.95mm_HandSolder
- R402: footprint Resistor_SMD:R_0805_2012Metric_Pad1.15x1.40mm_HandSolder -> Resistor_SMD:R_0603_1608Metric_Pad0.98x0.95mm_HandSolder
Changed lines of the file:
@@
 F 0 "R401" H 3870 1646 50  0000 L CNN
 F 1 "100k" H 3870 1555 50  0000 L CNN
-F 2 "Resistor_SMD:R_0603_1608Metric_Pad1.05x0.95mm_HandSolder" V 3730 1600 50  0001 C CNN
+F 2 "Resistor_SMD:R_0603_1608Metric_Pad0.98x0.95mm_HandSolder" V 3730 1600 50  0001 C CNN
 F 3 "~" H 3800 1600 50  0001 C CNN
 	1    3800 1600
@@
 F 0 "R403" H 6520 1846 50  0000 L CNN
 F 1 "370" H 6520 1755 50  0000 L CNN
-F 2 "Resistor_SMD:R_0603_1608Metric_Pad1.05x0.95mm_HandSolder" V 6380 1800 50  0001 C CNN
+F 2 "Resistor_SMD:R_0603_1608Metric_Pad0.98x0.95mm_HandSolder" V 6380 1800 50  0001 C CNN
 F 3 "~" H 6450 1800 50  0001 C CNN
 	1    6450 1800
@@
 F 0 "R402" H 5970 1696 50  0000 L CNN
 F 1 "6k8/0.5W" H 5970 1605 50  0000 L CNN
-F 2 "Resistor_SMD:R_0805_2012Metric_Pad1.15x1.40mm_HandSolder" V 5830 1650 50  0001 C CNN
+F 2 "Resistor_SMD:R_0603_1608Metric_Pad0.98x0.95mm_HandSolder" V 5830 1650 50  0001 C CNN
 F 3 "~" H 5900 1650 50  0001 C CNN
 	1    5900 1650
@@
 F 0 "C405" H 6915 4796 50  0000 L CNN
 F 1 "100n" H 6915 4705 50  0000 L CNN
-F 2 "Capacitor_SMD:C_0603_1608Metric_Pad1.05x0.95mm_HandSolder" H 6838 4600 50  0001 C CNN
+F 2 "Capacitor_SMD:C_0603_1608Metric_Pad1.08x0.95mm_HandSolder" H 6838 4600 50  0001 C CNN
 F 3 "~" H 6800 4750 50  0001 C CNN
 	1    6800 4750
@@
 F 0 "C402" H 5115 4796 50  0000 L CNN
 F 1 "100n" H 5115 4705 50  0000 L CNN
-F 2 "Capacitor_SMD:C_0603_1608Metric_Pad1.05x0.95mm_HandSolder" H 5038 4600 50  0001 C CNN
+F 2 "Capacitor_SMD:C_0603_1608Metric_Pad1.08x0.95mm_HandSolder" H 5038 4600 50  0001 C CNN
 F 3 "~" H 5000 4750 50  0001 C CNN
 	1    5000 4750
