File: hardware/project/ETH6C20MUX/Ethernet.sch (KiCad schematic (older format))
At the start: 43 parts, among them U201 LC03-3.3, U202 LAN8742A, U203 LC03-3.3, Y201 NX5032GA-25.000M-LN-CD-1

Commit message: Updated PCB. Added 3D components. Started BOM list.
Parts:
- L201: footprint ETH6C16MXU:749010012A -> ETH6C20MUX:749010012A
- U201, U203: footprint ETH6C16MXU:SO8E -> ETH6C20MUX:SO8E
- Y201: footprint ETH6C16MXU:NX5032GA -> ETH6C20MUX:NX5032GA
Changed lines of the file:
@@
 F 0 "L201" H 8350 3765 50  0000 C CNN
 F 1 "749010012A" H 8350 3674 50  0000 C CNN
-F 2 "ETH6C16MXU:749010012A" H 9350 3450 50  0001 C CNN
+F 2 "ETH6C20MUX:749010012A" H 9350 3450 50  0001 C CNN
 F 3 "" H 9350 3450 50  0001 C CNN
 	1    8350 3200
@@
 F 0 "U201" H 10450 3287 60  0000 C CNN
 F 1 "LC03-3.3" H 10450 3181 60  0000 C CNN
-F 2 "ETH6C16MXU:SO8E" H 10450 2850 60  0001 C CNN
+F 2 "ETH6C20MUX:SO8E" H 10450 2850 60  0001 C CNN
 F 3 "" H 10450 2850 60  0000 C CNN
 	1    10450 2850
@@
 F 0 "U203" H 10450 4087 60  0000 C CNN
 F 1 "LC03-3.3" H 10450 3981 60  0000 C CNN
-F 2 "ETH6C16MXU:SO8E" H 10450 3650 60  0001 C CNN
+F 2 "ETH6C20MUX:SO8E" H 10450 3650 60  0001 C CNN
 F 3 "" H 10450 3650 60  0000 C CNN
 	1    10450 3650
@@
 F 0 "Y201" H 1900 4482 50  0000 C CNN
 F 1 "NX5032GA-25.000M-LN-CD-1" H 1900 4573 50  0000 C CNN
-F 2 "ETH6C16MXU:NX5032GA" H 1900 4750 50  0001 C CNN
+F 2 "ETH6C20MUX:NX5032GA" H 1900 4750 50  0001 C CNN
 F 3 "~" H 1900 4750 50  0001 C CNN
 	1    1900 4750

Commit message: PCB redesign
Parts:
- C201, C202, C203, C204, C205, C206, C207, C208, C209, C210, C213, C214: footprint Capacitor_SMD:C_0603_1608Metric_Pad1.05x0.95mm_HandSolder -> Capacitor_SMD:C_0603_1608Metric_Pad1.08x0.95mm_HandSolder
- D201: value YELLOW -> GREEN
- D202: value GREEN -> YELLOW
- R201, R202, R203, R204, R205, R206, R207, R208, R209, R210, R211, R212, R213, R214, R215, R217, R218, R219, R220, R221: footprint Resistor_SMD:R_0603_1608Metric_Pad1.05x0.95mm_HandSolder -> Resistor_SMD:R_0603_1608Metric_Pad0.98x0.95mm_HandSolder
- R216: footprint Resistor_SMD:R_1206_3216Metric_Pad1.42x1.75mm_HandSolder -> Resistor_SMD:R_0603_1608Metric_Pad0.98x0.95mm_HandSolder

Commit message: PCB design
Parts:
- R216: footprint Resistor_SMD:R_0603_1608Metric_Pad0.98x0.95mm_HandSolder -> Resistor_SMD:R_1206_3216Metric_Pad1.30x1.75mm_HandSolder
Changed lines of the file:
@@
 F 0 "R216" V 8143 4500 50  0000 C CNN
 F 1 "1M/1kV" V 8234 4500 50  0000 C CNN
-F 2 "Resistor_SMD:R_0603_1608Metric_Pad0.98x0.95mm_HandSolder" V 8280 4500 50  0001 C CNN
+F 2 "Resistor_SMD:R_1206_3216Metric_Pad1.30x1.75mm_HandSolder" V 8280 4500 50  0001 C CNN
 F 3 "~" H 8350 4500 50  0001 C CNN
 	1    8350 4500
